File: kicadFiles/shark.kicad_pcb (KiCad board)
At the start: 2 copper layers, 225.6 x 74.6 mm, 291 parts, among them J1 TYPE-C-31-M12_13, J2 ARM JTAG, Q1 DTC123JKAT146, Q2 AO3401A, Q3 DTC123JKAT146, Q4 MMBFJ270, SW1 ESC, SW10 O, SW11 P, SW12 BKSP, SW13 TAB, SW14 A, SW15 S, SW16 D, SW17 F, SW18 G, SW19 H, SW2 Q, SW20 J, SW21 K, SW22 L, SW23 COLON, SW24 QUOTE, SW25 SHIFT, SW26 Z, SW27 X, SW28 C, SW29 V, SW3 W, SW30 B, SW31 N, SW32 M, SW33 COMMA, SW34 DOT, SW35 SLSH, SW36 ENTER, SW37 CTRL, SW38 Q, SW39 WIN, SW4 E, SW40 ALT, SW41 F1, SW42 SPC_100, SW43 SPC_100, SW44 F2, SW45 LEFT, SW46 DOWN, SW47 UP, SW48 RIGHT, SW49 SPC_200, SW5 R, SW50 SPC_200, SW51 SPC_200, SW6 T, SW7 Y, SW8 U, SW9 I, U1 STM32F072CBT6, U2 USBLC6-2SC6, U3 MCP1700T-3302E/TT, U4 TXS0101

Commit message: Reset circuit, level translator, SWD
Parts:
- removed R63, R67, R69: 420R, acheron_Components:R_SMD_1206
- R61: value 420R -> 10k
- moved C16 235.4 mm to (251.6, 71.1), turned to 90 degrees
- moved R61 211.1 mm to (256.5, 77.8), turned to 180 degrees
- moved Q2 209.6 mm to (267.2, 87.3), turned to 90 degrees
- moved C15 207.4 mm to (252.3, 77.4), turned to 90 degrees
- moved U4 188.6 mm to (255.6, 74.5), turned to 90 degrees
- moved Q3 188.5 mm to (270.4, 102.9)
- moved R13 161.7 mm to (269.2, 106.1)
- moved R12 160.8 mm to (265.9, 103.5), turned to 180 degrees
- moved R9 106.9 mm to (261.6, 97.2), turned to 90 degrees
- moved Q4 102.7 mm to (240.0, 126.5), turned to 90 degrees
- moved R77 102.4 mm to (235.1, 126.0)
- moved R11 97.1 mm to (248.5, 124.5), turned to 90 degrees
- moved R10 95.8 mm to (251.2, 124.5), turned to 90 degrees
- moved D52 90.8 mm to (253.9, 127.5), turned to -90 degrees
- moved Q1 82.3 mm to (257.7, 128.1), turned to 90 degrees
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Connections:
- R61 pad 1: (no net) -> Net-(R61-Pad1)
- R61 pad 2: Net-(Q2-Pad3) -> 3V3
- U4 pad 5: 3V3 -> Net-(R61-Pad1)
Routing:
- net 3V3: track 39.0 -> 160.2 mm, vias 6 -> 11
- net 5V: track 14.9 -> 69.2 mm, vias 0 -> 2
- net NRST: track 0.00 -> 45.8 mm
- net RGB_3V3: track 0.00 -> 38.9 mm, vias 0 -> 2
- net LED_PWM: track 0.00 -> 34.7 mm
- net SWDIO: track 0.00 -> 33.7 mm
- net Net-(Q2-Pad3): track 1068.5 -> 1035.3 mm
- net SWCLK: track 0.00 -> 31.8 mm
- net Net-(D52-Pad2): track 0.00 -> 28.6 mm, vias 0 -> 2
- net Net-(Q2-Pad1): track 0.00 -> 27.4 mm, vias 0 -> 2
- net RGB_5V: track 0.00 -> 25.5 mm
- net BOOT0: track 0.00 -> 19.1 mm
- net Net-(Q3-Pad3): track 0.00 -> 8.51 mm
- net C0: track 66.1 -> 73.7 mm
- net Net-(D38-Pad2): track 4.87 -> 12.5 mm
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Other:
- board text added: "CLK"
- board text added: "IO"
- board text added: "SWD"
