File: kicadFiles/shark.kicad_sch (KiCad schematic)
At the start: 287 parts, among them J1 TYPE-C-31-M12_13, J2 ARM JTAG, Q1 DTC123JKAT146, Q2 AO3401A, Q3 DTC123JKAT146, Q4 MMBFJ270, SW1 ESC, SW10 O, SW11 P, SW12 BKSP, SW13 TAB, SW14 A, SW15 S, SW16 D, SW17 F, SW18 G, SW19 H, SW2 Q, SW20 J, SW21 K, SW22 L, SW23 COLON, SW24 QUOTE, SW25 SHIFT, SW26 Z, SW27 X, SW28 C, SW29 V, SW3 W, SW30 B, SW31 N, SW32 M, SW33 COMMA, SW34 DOT, SW35 SLSH, SW36 ENTER, SW37 CTRL, SW38 Q, SW39 WIN, SW4 E, SW40 ALT, SW41 F1, SW42 SPC_100, SW43 SPC_100, SW44 F2, SW45 LEFT, SW46 DOWN, SW47 UP, SW48 RIGHT, SW49 SPC_200, SW5 R, SW50 SPC_200, SW51 SPC_200, SW6 T, SW7 Y, SW8 U, SW9 I, U1 STM32F072CBT6, U2 USBLC6-2SC6, U3 MCP1700T-3302E/TT, U4 TXS0101

Commit message: Reset circuit, level translator, SWD
Parts:
- added R61: 10k, acheron_Components:R_SMD_1206, symbol Device:R
Connections:
- net 3V3: now also R61.2; no longer U4.5 (OE)
- new net: R61.1, U4.5 (OE)
