File: kicadFiles/shark.sch (KiCad schematic (older format))
At the start: 268 parts, among them J1 TYPE-C-31-M12_13, J2 Conn_01x04_Male, J3 Conn_01x04_Male, J4 Conn_01x04_Male, J5 Conn_01x06_Male, Q1 AO4406AL, SW1 MXSwitch, SW10 MXSwitch, SW11 MXSwitch, SW12 MXSwitch, SW13 MXSwitch, SW14 MXSwitch, SW15 MXSwitch, SW16 MXSwitch, SW17 MXSwitch, SW18 MXSwitch, SW19 MXSwitch, SW2 MXSwitch, SW20 MXSwitch, SW21 MXSwitch, SW22 MXSwitch, SW23 MXSwitch, SW24 MXSwitch, SW25 MXSwitch, SW26 MXSwitch, SW27 MXSwitch, SW28 MXSwitch, SW29 MXSwitch, SW3 MXSwitch, SW30 MXSwitch, SW31 MXSwitch, SW32 MXSwitch, SW33 MXSwitch, SW34 MXSwitch, SW35 MXSwitch, SW36 MXSwitch, SW37 MXSwitch, SW38 MXSwitch, SW39 MXSwitch, SW4 MXSwitch, SW40 MXSwitch, SW41 MXSwitch, SW42 MXSwitch, SW43 MXSwitch, SW44 MXSwitch, SW45 MXSwitch, SW46 MXSwitch, SW47 MXSwitch, SW48 MXSwitch, SW49 MXSwitch, SW5 MXSwitch, SW50 MXSwitch, SW51 MXSwitch, SW6 MXSwitch, SW7 MXSwitch, SW8 MXSwitch, SW9 MXSwitch, U1 STM32F303-LQFP48, U2 MCP1700-3302E_SOT23, U3 USBLC6-2SC6, Y1 8MHz

Commit message: cache
Parts:
- CA1, CB1, CESD1, CRST1, CRST2, CSH1, CSI1, CSO1, CUSB1, CVB1, CVB2, CVB3, CVB4, CVB5, CVB6, CX1, CX2: symbol Device:C_Small -> shark-rescue:C_Small-Device
- D1, D10, D11, D12, D13, D14, D15, D16, D17, D18, D19, D2, D20, D21, D22, D23, D24, D25, D26, D27, D28, D29, D3, D30, D31, D32, D33, D34, D35, D36, D37, D38, D39, D4, D40, D41, D42, D43, D44, D45, D46, D47, D48, D5, D6, D7, D8, D9, DESD1, DLDO1, DRST1: symbol Device:D -> shark-rescue:D-Device
- DF1: symbol Device:D_Schottky_Small -> shark-rescue:D_Schottky_Small-Device
- F1: symbol Device:Polyfuse_Small -> shark-rescue:Polyfuse_Small-Device
- H1, H2, H3, H5, H6, L1, L2, L3, L4, L5, L6: symbol Mechanical:MountingHole -> shark-rescue:MountingHole-Mechanical
- H4: symbol Mechanical:MountingHole_Pad -> shark-rescue:MountingHole_Pad-Mechanical
- J1: symbol acheronSymbols:TYPE-C-31-M12_13 -> shark-rescue:TYPE-C-31-M12_13-acheronSymbols
- J2, J3, J4: symbol Connector:Conn_01x04_Male -> shark-rescue:Conn_01x04_Male-Connector
- J5: symbol Connector:Conn_01x06_Male -> shark-rescue:Conn_01x06_Male-Connector
- LED1, LED10, LED11, LED12, LED13, LED14, LED15, LED16, LED17, LED18, LED19, LED2, LED20, LED21, LED22, LED23, LED24, LED25, LED26, LED27, LED28, LED29, LED3, LED30, LED31, LED32, LED33, LED34, LED35, LED36, LED37, LED38, LED39, LED4, LED40, LED41, LED42, LED43, LED44, LED45, LED46, LED47, LED48, LED49, LED5, LED50, LED51, LED6, LED7, LED8, LED9: symbol acheronSymbols:LED -> shark-rescue:LED-acheronSymbols
- Q1: symbol acheronSymbols:AO4406AL -> shark-rescue:AO4406AL-acheronSymbols
- QRST1: symbol Transistor_BJT:DTC123J -> shark-rescue:DTC123J-Transistor_BJT
- RA1, RA2, RB1, RB2, RCC1, RCC2, RDM1, RDP1, RL1, RL10, RL11, RL12, RL13, RL14, RL15, RL16, RL17, RL18, RL19, RL2, RL20, RL21, RL22, RL23, RL24, RL25, RL26, RL27, RL28, RL29, RL3, RL30, RL31, RL32, RL33, RL34, RL35, RL36, RL37, RL38, RL39, RL4, RL40, RL41, RL42, RL43, RL44, RL45, RL46, RL47, RL48, RL5, RL6, RL7, RL8, RL9, RPG1, RPU1, RRST1, RSG1: symbol Device:R_Small -> shark-rescue:R_Small-Device
- RESD1, RSH1: symbol Device:R -> shark-rescue:R-Device
- RGB1, RGB2, RGB3, RGB4, RGB5, RGB6, RGB7, RGB8: symbol LED:WS2812B -> shark-rescue:WS2812B-LED
- ROT1, ROT2: symbol Device:Rotary_Encoder_Switch -> shark-rescue:Rotary_Encoder_Switch-Device
- SRST1: symbol Switch:SW_Push -> shark-rescue:SW_Push-Switch
- SW1, SW10, SW11, SW12, SW13, SW14, SW15, SW16, SW17, SW18, SW19, SW2, SW20, SW21, SW22, SW23, SW24, SW25, SW26, SW27, SW28, SW29, SW3, SW30, SW31, SW32, SW33, SW34, SW35, SW36, SW37, SW38, SW39, SW4, SW40, SW41, SW42, SW43, SW44, SW45, SW46, SW47, SW48, SW49, SW5, SW50, SW51, SW6, SW7, SW8, SW9: symbol acheronSymbols:MXSwitch -> shark-rescue:MXSwitch-acheronSymbols
- U1: symbol acheronSymbols:STM32F303-LQFP48 -> shark-rescue:STM32F303-LQFP48-acheronSymbols
- U2: symbol Regulator_Linear:MCP1700-3302E_SOT23 -> shark-rescue:MCP1700-3302E_SOT23-Regulator_Linear
- U3: symbol Power_Protection:USBLC6-2SC6 -> shark-rescue:USBLC6-2SC6-Power_Protection
- Y1: symbol Device:Crystal_GND24 -> shark-rescue:Crystal_GND24-Device
